File: kicad/kicad.kicad_pcb (KiCad board)
At the start: 2 copper layers, 83.8 x 61 mm, 22 parts, among them J1 USB_A_MIDI, J2 LED_DATA, J3 POWER_CONNECTOR, J4 DMX_INPUT, J5 DMX_OUTPUT, SW2 SW_DIP_MODE_SWITCH, U1 Teensy4.0, U2 74AHCT125, U3 TPS2051BD, U4 MAX485_MODULE

Commit message: PicoAudio first commit
Other:
- net class Default removed
- net class Power removed
